File: PCBs/soccer bottom.kicad_sch (KiCad schematic)
At the start: 3 parts, among them U1 CD74HC4067SM, U2 QRE1113GR, U3 QRE1113GR

Commit message: v5
Parts:
- added J1: Conn_01x04_Socket, Connector_JST:JST_XH_B4B-XH-A_1x04_P2.50mm_Vertical, symbol Connector:Conn_01x04_Socket
- added J2: Conn_01x02_Socket, Connector_JST:JST_XH_B2B-XH-AM_1x02_P2.50mm_Vertical, symbol Connector:Conn_01x02_Socket
Connections:
- net at U1.10 (S0): now also J1.1 (Pin_1)
- net at U1.11 (S1): now also J1.2 (Pin_2)
- net GND: now reaches U1.12 (GND)
- net GND: now also J2.2 (Pin_2)
- net at U1.13 (S3): now also J1.4 (Pin_4)
- net at U1.14 (S2): now also J1.3 (Pin_3)
- net +5V: now reaches U1.24 (VCC)
- net +5V: now also J2.1 (Pin_1)

Commit message: test
Connections:
- net GND: now also U1.15 (~{E})
Changed lines of the file:
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@@
 	(generator_version "9.0")
 	(paper "A4")
+	(junction
+		(at 120.65 127)
+		(diameter 0)
+		(color 0 0 0 0)
+	)
 	(wire
 		(pts
-			(xy 120.65 124.46) (xy 120.65 130.81)
+			(xy 120.65 124.46) (xy 120.65 127)
+		)
+		(stroke
+			(width 0)
+			(type default)
+		)
+	)
+	(wire
+		(pts
+			(xy 107.95 127) (xy 120.65 127)
 		)
 		(stroke
@@
 		(pts
 			(xy 102.87 101.6) (xy 107.95 101.6)
+		)
+		(stroke
+			(width 0)
+			(type default)
+		)
+	)
+	(wire
+		(pts
+			(xy 107.95 111.76) (xy 107.95 127)
 		)
 		(stroke
@@
 		)
 		(stroke
+			(width 0)
+			(type default)
+		)
+	)
+	(wire
+		(pts
+			(xy 120.65 127) (xy 120.65 130.81)
+		)
+		(stroke

Commit message: e
Parts:
- removed J2: Conn_01x02_Socket, Connector_JST:JST_XH_B2B-XH-AM_1x02_P2.50mm_Vertical, symbol Connector:Conn_01x02_Socket
- added J2: Conn_01x03_Socket, Connector_JST:JST_XH_B3B-XH-A_1x03_P2.50mm_Vertical, symbol Connector:Conn_01x03_Socket
Connections:
- net +5V: now also J2.1 (Pin_1)
- net GND: now also J2.2 (Pin_2)
- net at U1.1 (COM): now also J2.3 (Pin_3)
Changed lines of the file:
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@@
+	(wire
+		(pts
+			(xy 102.87 78.74) (xy 102.87 76.2)
+		)
+		(stroke
+			(width 0)
+			(type default)
+		)
+	)
 	(wire
 		(pts
@@
 	(wire
 		(pts
+			(xy 97.79 81.28) (xy 107.95 81.28)
+		)
+		(stroke
+			(width 0)
+			(type default)
+		)
+	)
+	(wire
+		(pts
 			(xy 107.95 111.76) (xy 107.95 127)
 		)
@@
 	(wire
 		(pts
-			(xy 90.17 107.95) (xy 93.98 107.95)
-		)
-		(stroke
-			(width 0)
-			(type default)
-		)
-	)
-	(wire
-		(pts
 			(xy 102.87 99.06) (xy 107.95 99.06)
 		)
@@
 	(wire
 		(pts
-			(xy 90.17 110.49) (xy 93.98 110.49)
+			(xy 97.79 83.82) (xy 107.95 83.82)
+		)
+		(stroke
+			(width 0)
+			(type default)
+		)
+	)
+	(wire
+		(pts
+			(xy 97.79 78.74) (xy 102.87 78.74)
 		)
 		(stroke
@@
 	(symbol
 		(lib_id "power:+5V")
-		(at 93.98 107.95 0)
+		(at 102.87 76.2 0)
 		(unit 1)
 		(exclude_from_sim no)
@@
 		(dnp no)
 		(property "Reference" "#PWR03"
-			(at 93.98 111.76 0)
+			(at 102.87 80.01 0)
 			(effects
 				(font
@@
 		)
 		(property "Value" "+5V"
-			(at 93.98 103.124 0)
+			(at 102.87 71.374 0)
 			(effects
 				(font
@@
 		)
 		(property "Footprint" ""
-			(at 93.98 107.95 0)
+			(at 102.87 76.2 0)
 			(effects
 				(font
@@
 		)
 		(property "Datasheet" ""
-			(at 93.98 107.95 0)
+			(at 102.87 76.2 0)
 			(effects
 				(font
@@
 		)
 		(property "Description" "Power symbol creates a global label with name \"+5V\""
-			(at 93.98 107.95 0)
+			(at 102.87 76.2 0)
 			(effects
 				(font
@@
 	)
 	(symbol
-		(lib_id "Connector:Conn_01x02_Socket")
-		(at 85.09 107.95 0)
+		(lib_id "Connector:Conn_01x03_Socket")
+		(at 92.71 81.28 0)
 		(mirror y)
 		(unit 1)
@@
 		(dnp no)
 		(property "Reference" "J2"
-			(at 83.82 107.9499 0)
+			(at 91.44 80.0099 0)
 			(effects
 				(font
@@
 			)
 		)
-		(property "Value" "Conn_01x02_Socket"
-			(at 83.82 110.4899 0)
+		(property "Value" "Conn_01x03_Socket"
+			(at 91.44 82.5499 0)
 			(effects
 				(font
@@
 			)
 		)
-		(property "Footprint" "Connector_JST:JST_XH_B2B-XH-AM_1x02_P2.50mm_Vertical"
-			(at 85.09 107.95 0)
+		(property "Footprint" "Connector_JST:JST_XH_B3B-XH-A_1x03_P2.50mm_Vertical"
+			(at 92.71 81.28 0)
 			(effects
 				(font
@@
 		)
 		(property "Datasheet" "~"
-			(at 85.09 107.95 0)
-			(effects
-				(font
-					(size 1.27 1.27)
-				)
-				(hide yes)
-			)
-		)
-		(property "Description" "Generic connector, single row, 01x02, script generated"
-			(at 85.09 107.95 0)
-			(effects
-				(font
-					(size 1.27 1.27)
-				)
-				(hide yes)
-			)
+			(at 92.71 81.28 0)
+			(effects
+				(font
+					(size 1.27 1.27)
+				)
+				(hide yes)
+			)
+		)
+		(property "Description" "Generic connector, single row, 01x03, script generated"
+			(at 92.71 81.28 0)
+			(effects
+				(font
+					(size 1.27 1.27)
+				)
+				(hide yes)
+			)
+		)
+		(pin "3"
 		)
 		(pin "1"
@@
 	(symbol
 		(lib_id "power:GND")
-		(at 93.98 110.49 0)
-		(unit 1)
-		(exclude_from_sim no)
-		(in_bom yes)
-		(on_board yes)
-		(dnp no)
-		(fields_autoplaced yes)
+		(at 107.95 81.28 0)
+		(mirror x)
+		(unit 1)
+		(exclude_from_sim no)
+		(in_bom yes)
+		(on_board yes)
+		(dnp no)
 		(property "Reference" "#PWR05"
-			(at 93.98 116.84 0)
+			(at 107.95 74.93 0)
 			(effects
 				(font
@@
 		)
 		(property "Value" "GND"
-			(at 93.98 115.57 0)
+			(at 107.95 76.2 0)
 			(effects
 				(font
@@
 		)
 		(property "Footprint" ""
-			(at 93.98 110.49 0)
+			(at 107.95 81.28 0)
 			(effects
 				(font
@@
 		)
 		(property "Datasheet" ""
-			(at 93.98 110.49 0)
+			(at 107.95 81.28 0)
 			(effects
 				(font
@@
 		)
 		(property "Description" "Power symbol creates a global label with name \"GND\" , ground"
-			(at 93.98 110.49 0)
-			(effects
-				(font
+			(at 107.95 81.28 0)
+			(effects
+				(font

Commit message: r
Parts:
- removed U3: QRE1113GR, OptoDevice:OnSemi_CASE100CY, symbol Sensor_Proximity:QRE1113GR
- added R1: 100, Resistor_SMD:R_1206_3216Metric, symbol Device:R
- added R2: 10k, Resistor_SMD:R_0805_2012Metric, symbol Device:R
Connections:
- net +5V: now also R1.1, R2.1
- net GND: now also U2.2 (K), U2.4
- net ir_0: now reaches U1.9 (I0)
- net at U2.1 (A): now also R2.2
- net at U2.3: now also R1.2
Other:
- moved on the sheet: U2

Commit message: ee?
Parts:
- added R10, R12, R14, R16, R18, R20, R22, R24, R26, R28, R30, R32, R33, R4, R6, R8: 10k, Resistor_SMD:R_0805_2012Metric, symbol Device:R
- added R11, R13, R15, R17, R19, R21, R23, R25, R27, R29, R3, R31, R5, R7, R9: 100, Resistor_SMD:R_1206_3216Metric, symbol Device:R
- added U10, U11, U12, U13, U14, U15, U16, U17, U3, U4, U5, U6, U7, U8, U9: QRE1113GR, OptoDevice:OnSemi_CASE100CY, symbol Sensor_Proximity:QRE1113GR
Connections:
- net +5V: now also R10.1, R11.1, R12.1, R13.1, R14.1, R15.1, R16.1, R17.1, R18.1, R19.1, R20.1, R21.1, R22.1, R23.1, R24.1, R25.1, R26.1, R27.1, R28.1, R29.1, R3.1, R30.1, R31.1, R32.1, R4.1, R5.1, R6.1, R7.1, R8.1, R9.1
- net GND: now also R33.2, U10.2 (K), U10.4, U11.2 (K), U11.4, U12.2 (K), U12.4, U13.2 (K), U13.4, U14.2 (K), U14.4, U15.2 (K), U15.4, U16.2 (K), U16.4, U17.2 (K), U17.4, U3.2 (K), U3.4, U4.2 (K), U4.4, U5.2 (K), U5.4, U6.2 (K), U6.4, U7.2 (K), U7.4, U8.2 (K), U8.4, U9.2 (K), U9.4; no longer U1.15 (~{E})
- net ir_0: now also R1.2, U2.3
- net ir_15: now reaches U1.16 (I15)
- net ir_15: now also R31.2, U17.3
- net ir_14: now reaches U1.17 (I14)
- net ir_14: now also R29.2, U16.3
- net ir_13: now reaches U1.18 (I13)
- net ir_13: now also R27.2, U15.3
- net ir_12: now reaches U1.19 (I12)
- net ir_12: now also R25.2, U14.3
- net ir_7: now reaches U1.2 (I7)
- net ir_7: now also R15.2, U9.3
- net ir_11: now reaches U1.20 (I11)
- net ir_11: now also R23.2, U13.3
- net ir_10: now reaches U1.21 (I10)
- net ir_10: now also R21.2, U12.3
- net ir_9: now reaches U1.22 (I9)
- net ir_9: now also R19.2, U11.3
- net ir_8: now reaches U1.23 (I8)
- net ir_8: now also R17.2, U10.3
- net ir_6: now reaches U1.3 (I6)
- net ir_6: now also R13.2, U8.3
- net ir_5: now reaches U1.4 (I5)
- net ir_5: now also R11.2, U7.3
- net ir_4: now reaches U1.5 (I4)
- net ir_4: now also R9.2, U6.3
- net ir_3: now reaches U1.6 (I3)
- net ir_3: now also R7.2, U5.3
- net ir_2: now reaches U1.7 (I2)
- net ir_2: now also R5.2, U4.3
- net ir_1: now reaches U1.8 (I1)
- net ir_1: now also R3.2, U3.3
- new net: R8.2, U5.1 (A)
- new net: R28.2, U15.1 (A)
- new net: R6.2, U4.1 (A)
- new net: R24.2, U13.1 (A)
- new net: R16.2, U9.1 (A)
- new net: R4.2, U3.1 (A)
- new net: R20.2, U11.1 (A)
- new net: R33.1, U1.15 (~{E})
- new net: R26.2, U14.1 (A)
- new net: R32.2, U17.1 (A)
- new net: R18.2, U10.1 (A)
- new net: R22.2, U12.1 (A)
- new net: R30.2, U16.1 (A)
- new net: R12.2, U7.1 (A)
- new net: R10.2, U6.1 (A)
- new net: R14.2, U8.1 (A)
Other:
- moved on the sheet: J1, J2, R1, R2, U1, U2
