File: PCBs/soccer bottom.kicad_pcb (KiCad board)
At the start: 2 copper layers, 52 parts, among them J1 Conn_01x04_Socket, J2 Conn_01x03_Socket, U1 CD74HC4067SM, U10 QRE1113GR, U11 QRE1113GR, U12 QRE1113GR, U13 QRE1113GR, U14 QRE1113GR, U15 QRE1113GR, U16 QRE1113GR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

Commit message: eeee
Parts:
- J1, J2: moved to B.Cu
- moved R13 172.3 mm to (259.0, 62.5)
- moved R25 145.5 mm to (234.4, 79.0)
- moved U4 129.9 mm to (71.7, 128.3), turned to 45 degrees
- moved R11 129.3 mm to (209.0, 84.9)
- moved R2 129.3 mm to (189.1, 97.0)
- moved R26 129.3 mm to (202.4, 97.0)
- moved R27 129.3 mm to (220.2, 71.7)
- moved R28 129.3 mm to (202.4, 100.0)
- moved R29 129.3 mm to (220.2, 75.0)
- moved R3 129.3 mm to (209.0, 71.7)
- moved R30 129.3 mm to (202.4, 102.9)
- moved R31 129.3 mm to (220.2, 78.3)
- moved R32 129.3 mm to (202.4, 105.9)
- moved R4 129.3 mm to (189.1, 100.0)
- moved R5 129.3 mm to (209.0, 75.0)
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
Commit message: v10 or smting
Parts:
- removed the R31 at (220.2, 78.3)
- removed the R32 at (202.4, 105.9)
- added R1: 100, Resistor_SMD:R_1206_3216Metric, F.Cu at (102.0, 133.2)
- added R2: 10k, Resistor_SMD:R_0805_2012Metric, F.Cu at (98.0, 133.2)
- moved R13 184.5 mm to (75.1, 78.0), turned to 135 degrees
- moved R9 143.6 mm to (66.8, 102.0), turned to 180 degrees
- moved R7 143.5 mm to (70.1, 114.5), turned to -157.5 degrees
- moved R11 140.5 mm to (68.6, 89.2), turned to 157.5 degrees
- moved R5 140.2 mm to (78.0, 124.9), turned to -135 degrees
- moved R3 133.9 mm to (89.2, 131.4), turned to -112.5 degrees
- moved R15 129.2 mm to (85.5, 70.1), turned to 112.5 degrees
- moved R10 126.7 mm to (66.8, 98.0), turned to 180 degrees
- moved R12 124.2 mm to (70.1, 85.5), turned to 157.5 degrees
- moved R8 120.6 mm to (68.6, 110.8), turned to -157.5 degrees
- moved R14 118.9 mm to (78.0, 75.1), turned to 135 degrees
- moved R17 116.9 mm to (98.0, 66.8), turned to 90 degrees
- moved R6 115.6 mm to (75.1, 122.0), turned to -135 degrees
- moved R16 110.8 mm to (89.2, 68.6), turned to 112.5 degrees
- moved R4 107.9 mm to (85.5, 129.9), turned to -112.5 degrees
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- renumbered R1 to R31, R2 to R32
Connections:
- R31 pad 2: /ir_0 -> /ir_15
- R32 pad 2: Net-(U2-A) -> Net-(U17-A)

Commit message: 20/2/26 test 1 final
Parts:
- turned R23 to 23 degrees
- turned R31 to -67 degrees
- turned R15 to 113 degrees
- turned R7 to -157 degrees
- turned R28 to -22 degrees
- turned R4 to -112 degrees
- turned R12 to 158 degrees
- turned R20 to 68 degrees
- turned U11 to -112 degrees
- turned U5 to 23 degrees
- turned U7 to -22 degrees
- turned U9 to -67 degrees
- turned U13 to -157 degrees
- turned U15 to 158 degrees
- turned U17 to 113 degrees
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Routing:
- net GND: track 0.00 -> 364.4 mm, vias 0 -> 2
- net +5V: track 0.00 -> 262.9 mm
- net /ir_7: track 0.00 -> 68.8 mm, vias 0 -> 2
- net /ir_6: track 0.00 -> 63.6 mm, vias 0 -> 2
- net /ir_2: track 0.00 -> 63.3 mm, vias 0 -> 2
- net /ir_1: track 0.00 -> 60.8 mm, vias 0 -> 2
- net /ir_3: track 0.00 -> 58.7 mm, vias 0 -> 2
- net /ir_8: track 0.00 -> 56.8 mm, vias 0 -> 2
- net /ir_5: track 0.00 -> 55.5 mm
- net /ir_4: track 0.00 -> 54.7 mm
- net /ir_0: track 0.00 -> 46.3 mm, vias 0 -> 2
- net /ir_15: track 0.00 -> 42.9 mm, vias 0 -> 2
- net /ir_9: track 0.00 -> 42.0 mm, vias 0 -> 2
- net /ir_10: track 0.00 -> 36.1 mm, vias 0 -> 2
- net /ir_14: track 0.00 -> 32.7 mm, vias 0 -> 2
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Other:
- board outline added: 90 x 90 mm
