File: PCBs/boost/boost/boost.kicad_sch (KiCad schematic)
At the start: 13 parts, among them Q1 TIP42A, Q2 BC547, Q3 BC547, Q4 BC547, Q5 BC547

Commit message: delete
Parts:
- removed C1: C_Polarized, symbol Device:C_Polarized
- removed D1: 1N4007, Diode_THT:D_DO-41_SOD81_P10.16mm_Horizontal, symbol Diode:1N4007
- removed Q1: TIP42A, Package_TO_SOT_THT:TO-220-3_Vertical, symbol Transistor_BJT:TIP42A
- removed Q2, Q3, Q4, Q5: BC547, Package_TO_SOT_THT:TO-92_Inline, symbol Transistor_BJT:BC547
- removed R1: 2.2k, symbol Device:R
- removed R2: 220, symbol Device:R
- removed R3, R4, R5, R6: 1k, symbol Device:R
