File: PCBs/kicker/kicker.kicad_sch (KiCad schematic)
At the start: 30 parts, among them J2 Conn_01x04_Socket, J3 Conn_01x01_Socket, J4 Conn_01x01_Socket, Q1 CSD19534Q5A, U1 UCC27624DR, U2 XL6019E1

Commit message: kicker V1
Parts:
- added R9: 3k, Resistor_SMD:R_2512_6332Metric, symbol Device:R
- added TP1: 48V probe, TestPoint:TestPoint_THTPad_1.5x1.5mm_Drill0.7mm, symbol Connector:TestPoint_Probe
- added TP2: GND probe, TestPoint:TestPoint_THTPad_1.5x1.5mm_Drill0.7mm, symbol Connector:TestPoint_Probe
- C3, C4, C5, C6: now not fitted
- J2: footprint Connector_JST:JST_XH_S4B-XH-A-1_1x04_P2.50mm_Horizontal -> Connector_JST:JST_XH_B4B-XH-A_1x04_P2.50mm_Vertical; now not fitted; now left out of the parts list
- U1: footprint SOIC127P599X175-8N -> Package_SO:SOIC-8_3.9x4.9mm_P1.27mm
Connections:
- net 48V+: now also TP1.1
- net GND: now also R9.2, TP2.1; no longer J4.1 (Pin_1)
- net SOLin: now reaches C3.1, C4.1, C5.1, C6.1, R5.2
- net SOLin: now also J4.1 (Pin_1), R9.1

Commit message: kicker v2 review
Other:
- moved on the sheet: C1, C2, C3, C4, C5, C6, J2, J3, J4, Q1, R1, R2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
