File: PCBs/kicker/kicker.kicad_sch (KiCad schematic)
At the start: 33 parts, among them J2 Conn_01x04_Socket, J3 Conn_01x01_Socket, J4 Conn_01x01_Socket, Q1 CSD19534Q5A, U1 UCC27624DR, U2 XL6019E1

Commit message: kicker v2
Parts:
- added H1: MountingHole, MountingHole:MountingHole_3.2mm_M3, symbol Mechanical:MountingHole
- J3, J4: footprint Connector_Wire:SolderWirePad_1x01_SMD_5x10mm -> Connector_Wire:SolderWirePad_1x01_SMD_3x6mm
Changed lines of the file:
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@@
 			)
 		)
-		(property "Footprint" "Connector_Wire:SolderWirePad_1x01_SMD_5x10mm"
+		(property "Footprint" "Connector_Wire:SolderWirePad_1x01_SMD_3x6mm"
 			(at 229.87 43.18 0)
 			(effects
@@
 	)
 	(symbol
+		(lib_id "Mechanical:MountingHole")
+		(at 213.36 97.79 0)
+		(unit 1)
+		(exclude_from_sim no)
+		(in_bom no)
+		(on_board yes)
+		(dnp no)
+		(fields_autoplaced yes)
+		(property "Reference" "H1"
+			(at 215.9 96.5199 0)
+			(effects
+				(font
+					(size 1.27 1.27)
+				)
+				(justify left)
+			)
+		)
+		(property "Value" "MountingHole"
+			(at 215.9 99.0599 0)
+			(effects
+				(font
+					(size 1.27 1.27)
+				)
+				(justify left)
+			)
+		)
+		(property "Footprint" "MountingHole:MountingHole_3.2mm_M3"
+			(at 213.36 97.79 0)
+			(effects
+				(font
+					(size 1.27 1.27)
+				)
+				(hide yes)
+			)
+		)
+		(property "Datasheet" "~"
+			(at 213.36 97.79 0)
+			(effects
+				(font
+					(size 1.27 1.27)
+				)
+				(hide yes)
+			)
+		)
+		(property "Description" "Mounting Hole without connection"
+			(at 213.36 97.79 0)
+			(effects
+				(font
+					(size 1.27 1.27)
+				)
+				(hide yes)
+			)
+		)
+		(instances
+			(project ""
+				(path "/6b690c8d-b1b2-43bd-b6c1-471fc1941926"
+					(reference "H1")
+					(unit 1)
+				)
+			)
+		)
+	)
+	(symbol
 		(lib_id "Device:C_Polarized")
 		(at 157.48 97.79 0)
@@
 			)
 		)
-		(property "Footprint" "Connector_Wire:SolderWirePad_1x01_SMD_5x10mm"
+		(property "Footprint" "Connector_Wire:SolderWirePad_1x01_SMD_3x6mm"
 			(at 229.87 38.1 0)
 			(effects

Commit message: kicker fix
Changed lines of the file:
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@@
-	(wire
-		(pts
-			(xy 92.71 64.77) (xy 92.71 63.5)
-		)
-		(stroke
-			(width 0)
-			(type default)
-		)
-	)
 	(wire
 		(pts
@@
 	(wire
 		(pts
-			(xy 92.71 63.5) (xy 87.63 63.5)
+			(xy 87.63 63.5) (xy 93.98 63.5)
 		)
 		(stroke
@@
 		(pts
 			(xy 71.12 63.5) (xy 71.12 69.85)
-		)
-		(stroke
-			(width 0)
-			(type default)
-		)
-	)
-	(wire
-		(pts
-			(xy 92.71 64.77) (xy 93.98 64.77)
 		)
 		(stroke
@@
 	)
 	(label "capEN"
-		(at 93.98 64.77 0)
-		(effects
-			(font
+		(at 93.98 63.5 0)
+		(effects
+			(font

Commit message: e
Parts:
- R1, R8: value 2 -> 10
Changed lines of the file:
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@@
 			)
 		)
-		(property "Value" "2"
+		(property "Value" "10"
 			(at 106.172 114.3 90)
 			(show_name no)
@@
 			)
 		)
-		(property "Value" "2"
+		(property "Value" "10"
 			(at 106.172 109.22 90)
 			(show_name no)

Commit message: kicker rotate diode
Parts:
- removed D2: SS210, Diode_SMD:D_SMA, symbol Device:D_Schottky
Connections:
- net 48V+: now also C10.1, C9.1, D1.1 (K), R11.1
Other:
- moved on the sheet: TP1
Changed lines of the file:
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@@
 	)
 	(junction
-		(at 144.78 43.18)
+		(at 130.81 43.18)
+		(diameter 0)
+		(color 0 0 0 0)
+	)
+	(junction
+		(at 134.62 43.18)
 		(diameter 0)
 		(color 0 0 0 0)
@@
 	)
 	(junction
-		(at 130.81 43.18)
-		(diameter 0)
-		(color 0 0 0 0)
-	)
-	(junction
 		(at 149.86 93.98)
 		(diameter 0)
@@
 	(wire
 		(pts
-			(xy 71.12 59.69) (xy 71.12 53.34)
+			(xy 134.62 43.18) (xy 130.81 43.18)
 		)
 		(stroke
@@
 	(wire
 		(pts
-			(xy 59.69 119.38) (xy 59.69 124.46)
+			(xy 71.12 59.69) (xy 71.12 53.34)
 		)
 		(stroke
@@
 	(wire
 		(pts
-			(xy 130.81 69.85) (xy 135.89 69.85)
+			(xy 59.69 119.38) (xy 59.69 124.46)
 		)
 		(stroke
@@
 	(wire
 		(pts
-			(xy 87.63 140.97) (xy 87.63 139.7)
+			(xy 130.81 69.85) (xy 135.89 69.85)
 		)
 		(stroke
@@
 	(wire
 		(pts
-			(xy 144.78 38.1) (xy 144.78 43.18)
+			(xy 87.63 140.97) (xy 87.63 139.7)
 		)
 		(stroke
@@
 	(wire
 		(pts
+			(xy 130.81 43.18) (xy 130.81 49.53)
+		)
+		(stroke
+			(width 0)
+			(type default)
+		)
+	)
+	(wire
+		(pts
 			(xy 234.95 48.26) (xy 236.22 48.26)
 		)
@@
 	(wire
 		(pts
+			(xy 134.62 43.18) (xy 137.16 43.18)
+		)
+		(stroke
+			(width 0)
+			(type default)
+		)
+	)
+	(wire
+		(pts
 			(xy 134.62 93.98) (xy 135.89 93.98)
 		)
@@
 	(wire
 		(pts
-			(xy 130.81 43.18) (xy 134.62 43.18)
-		)
-		(stroke
-			(width 0)
-			(type default)
-		)
-	)
-	(wire
-		(pts
 			(xy 142.24 100.33) (xy 142.24 101.6)
 		)
@@
 	(wire
 		(pts
+			(xy 134.62 38.1) (xy 134.62 43.18)
+		)
+		(stroke
+			(width 0)
+			(type default)
+		)
+	)
+	(wire
+		(pts
 			(xy 68.58 43.18) (xy 49.53 43.18)
 		)
@@
 	(wire
 		(pts
-			(xy 130.81 49.53) (xy 130.81 43.18)
-		)
-		(stroke
-			(width 0)
-			(type default)
-		)
-	)
-	(wire
-		(pts
 			(xy 59.69 149.86) (xy 67.31 149.86)
 		)
@@
 	(wire
 		(pts
-			(xy 144.78 43.18) (xy 146.05 43.18)
-		)
-		(stroke
-			(width 0)
-			(type default)
-		)
-	)
-	(wire
-		(pts
 			(xy 172.72 93.98) (xy 180.34 93.98)
 		)
@@
 	(wire
 		(pts
-			(xy 142.24 43.18) (xy 144.78 43.18)
-		)
-		(stroke
-			(width 0)
-			(type default)
-		)
-	)
-	(wire
-		(pts
 			(xy 67.31 132.08) (xy 67.31 149.86)
 		)
@@
 	)
 	(label "48V+"
-		(at 146.05 43.18 0)
+		(at 137.16 43.18 0)
 		(effects
 			(font
@@
 	)
 	(symbol
-		(lib_id "Device:D_Schottky")
-		(at 138.43 43.18 0)
-		(mirror y)
-		(unit 1)
-		(body_style 1)
-		(exclude_from_sim no)
-		(in_bom yes)
-		(on_board yes)
-		(in_pos_files yes)
-		(dnp no)
-		(property "Reference" "D2"
-			(at 138.7475 36.83 0)
-			(show_name no)
-			(do_not_autoplace no)
-			(effects
-				(font
-					(size 1.27 1.27)
-				)
-			)
-		)
-		(property "Value" "SS210"
-			(at 138.7475 39.37 0)
-			(show_name no)
-			(do_not_autoplace no)
-			(effects
-				(font
-					(size 1.27 1.27)
-				)
-			)
-		)
-		(property "Footprint" "Diode_SMD:D_SMA"
-			(at 138.43 43.18 0)
-			(hide yes)
-			(show_name no)
-			(do_not_autoplace no)
-			(effects
-				(font
-					(size 1.27 1.27)
-				)
-			)
-		)
-		(property "Datasheet" ""
-			(at 138.43 43.18 0)
-			(hide yes)
-			(show_name no)
-			(do_not_autoplace no)
-			(effects
-				(font
-					(size 1.27 1.27)
-				)
-			)
-		)
-		(property "Description" "Schottky diode"
-			(at 138.43 43.18 0)
-			(hide yes)
-			(show_name no)
-			(do_not_autoplace no)
-			(effects
-				(font
-					(size 1.27 1.27)
-				)
-			)
-		)
-		(pin "1"
-		)
-		(pin "2"
-		)
-		(instances
-			(project "kicker"
-				(path "/6b690c8d-b1b2-43bd-b6c1-471fc1941926"
-					(reference "D2")
-					(unit 1)
-				)
-			)
-		)
-	)
-	(symbol
 		(lib_id "UCC27624DR:UCC27624DR")
 		(at 83.82 116.84 0)
@@
 	(symbol
 		(lib_id "Connector:TestPoint_Probe")
-		(at 144.78 38.1 0)
+		(at 134.62 38.1 0)
 		(unit 1)
 		(body_style 1)
@@
 		(fields_autoplaced yes)
 		(property "Reference" "TP1"
-			(at 148.59 35.2424 0)
+			(at 138.43 35.2424 0)
 			(show_name no)
 			(do_not_autoplace no)
@@
 		)
 		(property "Value" "48V probe"
-			(at 148.59 37.7824 0)
+			(at 138.43 37.7824 0)
 			(show_name no)
 			(do_not_autoplace no)
@@
 		)
 		(property "Footprint" "TestPoint:TestPoint_THTPad_1.5x1.5mm_Drill0.7mm"
-			(at 149.86 38.1 0)
+			(at 139.7 38.1 0)
 			(hide yes)
 			(show_name no)
@@
 		)
 		(property "Datasheet" ""
-			(at 149.86 38.1 0)
+			(at 139.7 38.1 0)
 			(hide yes)
 			(show_name no)
@@
 		)
 		(property "Description" "test point (alternative probe-style design)"
-			(at 144.78 38.1 0)
+			(at 134.62 38.1 0)
 			(hide yes)
 			(show_name no)

Commit message: kicker update
Parts:
- removed J2: Conn_01x04_Socket, Connector_JST:JST_XH_B4B-XH-A_1x04_P2.50mm_Vertical, symbol Connector:Conn_01x04_Socket
- added J1, J2: Screw_Terminal_01x02, TerminalBlock_Phoenix:TerminalBlock_Phoenix_MKDS-1,5-2_1x02_P5.00mm_Horizontal, symbol Connector:Screw_Terminal_01x02
Connections:
- net GND: now also J2.2 (Pin_2)
- net VCC: now also J2.1 (Pin_1)
- net mcuCap: now also J1.1 (Pin_1)
- net mcuKick: now also J1.2 (Pin_2)
Other:
- moved on the sheet: J3, J4

Commit message: main update
Parts:
- removed H1: MountingHole, MountingHole:MountingHole_3.2mm_M3, symbol Mechanical:MountingHole
- added H1: MountingHole_Pad, MountingHole:MountingHole_3.2mm_M3_DIN965_Pad, symbol Mechanical:MountingHole_Pad
- added H2, H3, H4: MountingHole_Pad, MountingHole_3.2mm_M3_DIN965_Pad, symbol Mechanical:MountingHole_Pad
- J1, J2: now not fitted; now left out of the parts list
Connections:
- net GND: now also H1.1, H2.1, H3.1, H4.1
Other:
- note added: "mounting holes"

Commit message: FINAL?
Parts:
- added D2: UF4007, Diode_THT:D_DO-41_SOD81_P10.16mm_Horizontal, symbol Device:D
Connections:
- net SOLin: now also D2.1 (K)
- net SOLout: now also D2.2 (A)
Changed lines of the file:
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@@
 	(rectangle
 		(start 207.01 33.02)
-		(end 233.68 59.69)
+		(end 241.3 59.69)
 		(stroke
 			(width 0)
@@
 	(wire
 		(pts
+			(xy 227.33 39.37) (xy 219.71 39.37)
+		)
+		(stroke
+			(width 0)
+			(type default)
+		)
+	)
+	(wire
+		(pts
 			(xy 130.81 69.85) (xy 135.89 69.85)
 		)
@@
 	(wire
 		(pts
+			(xy 227.33 36.83) (xy 227.33 39.37)
+		)
+		(stroke
+			(width 0)
+			(type default)
+		)
+	)
+	(wire
+		(pts
 			(xy 101.6 149.86) (xy 101.6 127)
 		)
@@
 	(wire
 		(pts
+			(xy 219.71 39.37) (xy 219.71 38.1)
+		)
+		(stroke
+			(width 0)
+			(type default)
+		)
+	)
+	(wire
+		(pts
 			(xy 83.82 149.86) (xy 87.63 149.86)
 		)
@@
 	(wire
 		(pts
+			(xy 229.87 36.83) (xy 227.33 36.83)
+		)
+		(stroke
+			(width 0)
+			(type default)
+		)
+	)
+	(wire
+		(pts
 			(xy 110.49 54.61) (xy 110.49 59.69)
 		)
@@
 	(wire
 		(pts
+			(xy 229.87 44.45) (xy 219.71 44.45)
+		)
+		(stroke
+			(width 0)
+			(type default)
+		)
+	)
+	(wire
+		(pts
 			(xy 106.68 59.69) (xy 106.68 62.23)
 		)
@@
 	(wire
 		(pts
+			(xy 219.71 44.45) (xy 219.71 43.18)
+		)
+		(stroke
+			(width 0)
+			(type default)
+		)
+	)
+	(wire
+		(pts
 			(xy 157.48 101.6) (xy 165.1 101.6)
 		)
@@
 					(unit 1)
 				)
+			)
+		)
+	)
+	(symbol
+		(lib_id "Device:D")
+		(at 229.87 40.64 270)
+		(unit 1)
+		(body_style 1)
+		(exclude_from_sim no)
+		(in_bom yes)
+		(on_board yes)
+		(in_pos_files yes)
+		(dnp no)
+		(fields_autoplaced yes)
+		(property "Reference" "D2"
+			(at 232.41 39.3699 90)
+			(show_name no)
+			(do_not_autoplace no)
+			(effects
+				(font
+					(size 1.27 1.27)
+				)
+				(justify left)
+			)
+		)
+		(property "Value" "UF4007"
+			(at 232.41 41.9099 90)
+			(show_name no)
+			(do_not_autoplace no)
+			(effects
+				(font
+					(size 1.27 1.27)
+				)
+				(justify left)
+			)
+		)
+		(property "Footprint" "Diode_THT:D_DO-41_SOD81_P10.16mm_Horizontal"
+			(at 229.87 40.64 0)
+			(hide yes)
+			(show_name no)
+			(do_not_autoplace no)
+			(effects
+				(font
+					(size 1.27 1.27)
+				)
+			)
+		)
+		(property "Datasheet" ""
+			(at 229.87 40.64 0)
+			(hide yes)
+			(show_name no)
+			(do_not_autoplace no)
+			(effects
+				(font
+					(size 1.27 1.27)
+				)
+			)
+		)
+		(property "Description" "Diode"
+			(at 229.87 40.64 0)
+			(hide yes)
+			(show_name no)
+			(do_not_autoplace no)
+			(effects
+				(font
+					(size 1.27 1.27)
+				)
+			)
+		)
+		(property "Sim.Device" "D"
+			(at 229.87 40.64 0)
+			(hide yes)
+			(show_name no)
+			(do_not_autoplace no)
+			(effects
+				(font
+					(size 1.27 1.27)
+				)
+			)
+		)
+		(property "Sim.Pins" "1=K 2=A"
+			(at 229.87 40.64 0)
+			(hide yes)
+			(show_name no)
+			(do_not_autoplace no)
+			(effects
+				(font
+					(size 1.27 1.27)
+				)
+			)
+		)
+		(pin "2"
+		)
+		(pin "1"
+		)
+		(instances
+			(project "kicker"
+				(path "/6b690c8d-b1b2-43bd-b6c1-471fc1941926"
+					(reference "D2")
+					(unit 1)
+				)
