File: PCBs/kicker/kicker.kicad_pcb (KiCad board)
At the start: 2 copper layers, 81.5 x 81.6 mm, 37 parts, among them J2 Conn_01x04_Socket, J3 Conn_01x01_Socket, J4 Conn_01x01_Socket, Q1 CSD19534Q5A, U1 UCC27624DR, U2 XL6019E1

Commit message: kicker v2 review
Parts:
- added G***: LOGO, LOGO, B.Cu at (154.2, 87.2)
Routing:
- net /SOLin: track 98.3 -> 108.5 mm
- net GND: vias 70 -> 89
Other:
- board text added: "MINDSTORMERS __/__/2026 kicker/boost pcb v1 designed by ___"
- board text added: "if you smell burning and look here, definitely wasn't my fault..."
- board text added: "pray to the electronics gods"

Commit message: kicker v2
Parts:
- J3, J4: footprint Connector_Wire:SolderWirePad_1x01_SMD_5x10mm -> Connector_Wire:SolderWirePad_1x01_SMD_3x6mm
- moved Q1 18.3 mm to (130.6, 118.7), turned to 180 degrees
- moved R4 17.6 mm to (135.0, 103.0), turned to 90 degrees
- moved R2 15.2 mm to (133.0, 103.0), turned to 90 degrees
- moved R1 14.9 mm to (133.5, 114.0), turned to -90 degrees
- moved R6 12.5 mm to (130.5, 103.0), turned to 90 degrees
- moved R8 11.4 mm to (130.5, 114.0), turned to -90 degrees
- moved U1 11.1 mm to (132.0, 108.3), turned to -90 degrees
- moved J4 11.0 mm to (140.0, 114.2)
- moved J3 10.9 mm to (124.8, 114.5), turned to 180 degrees
- moved R7 10.6 mm to (128.5, 103.0), turned to 90 degrees
- moved R3 9.16 mm to (135.5, 114.0), turned to 90 degrees
- moved C4 6.02 mm to (139.8, 125.2), turned to -90 degrees
- moved C2 5.48 mm to (128.0, 108.3), turned to 90 degrees
- moved C6 3.05 mm to (152.7, 115.7), turned to -45 degrees
- moved D1 2.83 mm to (152.8, 79.2)
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Routing:
- net /SOLin: track 108.5 -> 30.8 mm
- net VCC: track 67.3 -> 89.1 mm
- net Net-(D1-A): track 9.15 -> 30.2 mm
- net Net-(D1-K): track 17.4 -> 32.7 mm
- net /mcuKick: track 14.5 -> 25.4 mm
- net /capEN: track 37.6 -> 44.5 mm, vias 4 -> 3
- net /SOLout: track 12.4 -> 6.45 mm
- net /mcuCap: track 17.7 -> 21.2 mm
- net /outFET: track 6.55 -> 3.95 mm
- net GND: track 13.1 -> 10.5 mm, vias 89 -> 78
- net /48V+: track 37.1 -> 36.3 mm
- removed copper zone on F.Cu, net /capEN
- removed copper zone on F.Cu, net Net-(D1-A)
- removed copper zone on F.Cu, net VCC
Other:
- board text added: "GWSC 19/4/26 MINDSTORMERS 16V to 48V boost solenoid kicker designed by aiden"

Commit message: kicker v2.1
Other:
- board text added: "MINDSTORMERS 19/4/2026 kicker/boost pcb v2 designed by aiden"
- board text removed: "MINDSTORMERS __/__/2026 kicker/boost pcb v1 designed by ___"
