File: PCBs/middle/middle/middle.kicad_sch (KiCad schematic)
At the start: 11 parts, among them J1 Conn_01x04_Socket, J2 Conn_01x04_Socket, J3 Conn_01x04_Socket, J4 Conn_01x04_Socket, J5 Conn_01x04_Socket, J6 Conn_01x04_Socket, J7 Conn_01x02_Socket, U1 DEV-16771, U2 4754

Commit message: middle v2
Parts:
- removed F2: Fuse, Fuse:Fuseholder_Clip-5x20mm_Schurter_OG_Lateral_P15.00x5.00mm_D1.3mm_Horizontal, symbol Device:Fuse
- added R1: 4.7k, Resistor_THT:R_Axial_DIN0207_L6.3mm_D2.5mm_P10.16mm_Horizontal, symbol Device:R
- added R2: 1k, Resistor_THT:R_Axial_DIN0207_L6.3mm_D2.5mm_P10.16mm_Horizontal, symbol Device:R
Connections:
- net 3.3V is gone; now on net +3.3V: U1.3.3V_1 (3.3V), U1.3.3V_2 (3.3V), U1.3.3V_3 (3.3V)
- net +5V: now also U1.VIN; no longer J5.2 (Pin_2)
- net GND: now also R2.2
- net VCC: now also R1.1
- net at F1.2: now also J5.2 (Pin_2); no longer U1.VIN
- net Vbat: now reaches U1.14 (A0)
- net Vbat: now also R1.2, R2.1
Other:
- note added: "Vbat sensing"
- moved on the sheet: J5, U1

Commit message: e
Other:
- note added: "OpenMV RT1062"
- note removed: "OpenMV rt1062"
Changed lines of the file:
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@@
 		)
 	)
-	(text "OpenMV rt1062"
+	(text "OpenMV RT1062"
 		(exclude_from_sim no)
-		(at 174.752 101.6 0)
+		(at 175.26 101.6 0)
 		(effects
 			(font

Commit message: middle revision
Parts:
- added C1: 220u, Capacitor_THT:CP_Radial_D10.0mm_P3.80mm, symbol Device:C_Polarized
- added H2, H3, H4, H5: MountingHole_Pad, MountingHole:MountingHole_3.2mm_M3_DIN965_Pad, symbol Mechanical:MountingHole_Pad
- added R4, R5, R6: 10k, Resistor_THT:R_Axial_DIN0204_L3.6mm_D1.6mm_P5.08mm_Horizontal, symbol Device:R
- added SW1, SW2, SW3: SW_Push, Button_Switch_THT:SW_PUSH_6mm_H5mm, symbol Switch:SW_Push
- added U3: RFM69HCW, RF_Module:HOPERF_RFM9XW_THT, symbol RF_Module:RFM69HCW
- added U4: DM-OLED096-636, Footprints:MODULE_DM-OLED096-636, symbol DM-OLED096-636:DM-OLED096-636
- R1, R2: footprint Resistor_THT:R_Axial_DIN0207_L6.3mm_D2.5mm_P10.16mm_Horizontal -> Resistor_THT:R_Axial_DIN0204_L3.6mm_D1.6mm_P5.08mm_Horizontal
Connections:
- net +3.3V: now also C1.1, SW1.1, SW2.1, SW3.1, U3.13 (3.3V), U4.2 (VCC_IN)
- net CHARGE: now also U1.28 (RX7); no longer U1.37 (CS3)
- net GND: now also C1.2, H2.1, H3.1, H4.1, H5.1, R4.2, R5.2, R6.2, U3.1 (GND), U3.10 (GND), U3.8 (GND), U4.1 (GND)
- net KICK: now also U1.29 (TX7); no longer U1.36 (CS2)
- net MISO: now also U3.2 (MISO)
- net MOSI: now also U3.3 (MOSI)
- net SCL1: now also U4.3 (SCL)
- net SCLK: now also U3.4 (SCK)
- net SDA1: now also U4.4 (SDA)
- net at U1.20 (A6): now also R4.1, SW1.2
- net at U1.21 (A7): now also R5.1, SW2.2
- net at U1.22 (A8): now also R6.1, SW3.2
- net RFMreset: now reaches U1.34 (RX8)
- net RFMreset: now also U3.6 (RESET)
- net RFM0: now reaches U1.35 (TX8)
- net RFM0: now also U3.14 (DIO0)
- new net NSS: U1.36 (CS2), U3.5 (NSS)
Other:
- note added: "RFM69HCW 915MHz transceiver"

Commit message: mainboard layout
Parts:
- removed J1, J2, J3, J4, J5, J6: Conn_01x04_Socket, Connector_JST:JST_XH_B4B-XH-A_1x04_P2.50mm_Vertical, symbol Connector:Conn_01x04_Socket
- removed J7: Conn_01x02_Socket, Connector_JST:JST_XH_B2B-XH-A_1x02_P2.50mm_Vertical, symbol Connector:Conn_01x02_Socket
- removed U4: DM-OLED096-636, Footprints:MODULE_DM-OLED096-636, symbol DM-OLED096-636:DM-OLED096-636
- added H6: MountingHole_Pad, MountingHole:MountingHole_3.2mm_M3_DIN965_Pad, symbol Mechanical:MountingHole_Pad
- added J15, J16, J17, J18, J19, J20, J21: Screw_Terminal_01x02, TerminalBlock_Phoenix:TerminalBlock_Phoenix_MKDS-1,5-2_1x02_P5.00mm_Horizontal, symbol Connector:Screw_Terminal_01x02
- added J2, J3, J4, J5: Screw_Terminal_01x03, TerminalBlock_Phoenix:TerminalBlock_Phoenix_MKDS-1,5-3_1x03_P5.00mm_Horizontal, symbol Connector:Screw_Terminal_01x03
Connections:
- net +5V: now also J16.2 (Pin_2), J4.2 (Pin_2)
- net CHARGE: now also J21.1 (Pin_1)
- net GND: now also H6.1, J16.1 (Pin_1), J18.1 (Pin_1), J18.2 (Pin_2), J20.2 (Pin_2), J4.3 (Pin_3)
- net KICK: now also J21.2 (Pin_2)
- net M1A: now also J15.1 (Pin_1)
- net M1B: now also J15.2 (Pin_2)
- net M2A: now also J3.1 (Pin_1)
- net M2B: now also J3.2 (Pin_2)
- net M3A: now also J3.3 (Pin_3)
- net M3B: now also J2.1 (Pin_1)
- net M4A: now also J2.2 (Pin_2)
- net M4B: now also J2.3 (Pin_3)
- net MISO: now also J5.2 (Pin_2)
- net MOSI: now also J5.1 (Pin_1)
- net SCL1: now also J17.1 (Pin_1)
- net SCLK: now also J5.3 (Pin_3)
- net SDA1: now also J17.2 (Pin_2)
- net SS: now also J4.1 (Pin_1)
- net VCC: now also J19.1 (Pin_1), J20.1 (Pin_1)
- net at F1.2: now also J19.2 (Pin_2)

Commit message: e
Parts:
- removed J20: Screw_Terminal_01x02, TerminalBlock_Phoenix:TerminalBlock_Phoenix_MKDS-1,5-2_1x02_P5.00mm_Horizontal, symbol Connector:Screw_Terminal_01x02
Connections:
- net GND: now also J19.2 (Pin_2); no longer J18.1 (Pin_1)
- net at F1.2: now also J18.1 (Pin_1); no longer J19.2 (Pin_2)

Commit message: middle BANANA board layout, wiring
Connections:
- net CHARGE: now also J21.2 (Pin_2); no longer J21.1 (Pin_1)
- net KICK: now also J21.1 (Pin_1); no longer J21.2 (Pin_2)
Changed lines of the file:
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@@
 	)
 	(label "CHARGE"
-		(at 180.34 44.45 180)
+		(at 180.34 46.99 180)
 		(effects
 			(font
@@
 	)
 	(label "KICK"
-		(at 180.34 46.99 180)
-		(effects
-			(font
+		(at 180.34 44.45 180)
+		(effects
+			(font

Commit message: main update
Connections:
- net SCL1: now also U2.JP1_4 (SCL); no longer J17.1 (Pin_1)
- net SDA1: now also U2.JP1_5 (SDA); no longer J17.2 (Pin_2)
- net Vbat: now also U1.16 (A2); no longer U1.14 (A0)
- net TX: now reaches U1.15 (A1)
- net TX: now also J17.1 (Pin_1)
- removed net SCL2: U1.16 (A2), U2.JP1_4 (SCL)
- net SDA2: no longer names the net of U1.17 (A3)
- net SDA2: no longer U2.JP1_5 (SDA)
- new net RX: J17.2 (Pin_2), U1.14 (A0)
Other:
- note added: "CONNECTIONS"
- note added: "LD14P LiDAR"
- note added: "ONBOARD SENSORS"
- note added: "TEENSY 4.1"
- note added: "mounting holes"
- note removed: "border detection board"
- moved on the sheet: C1, F1, H2, H3, H4, H5, H6, J15, J16, J17, J18, J19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

Commit message: nrf middle update 1 (NOT DONE)
Parts:
- removed U3: RFM69HCW, RF_Module:HOPERF_RFM9XW_THT, symbol RF_Module:RFM69HCW
- added U3: NRF24L01_Breakout, RF_Module:nRF24L01_Breakout, symbol RF:NRF24L01_Breakout
- C1: value 220u -> 100u; footprint Capacitor_THT:CP_Radial_D10.0mm_P3.80mm -> Capacitor_THT:CP_Radial_D6.3mm_P2.50mm
Connections:
- net +3.3V: now also U3.2 (VCC)
- net GND: now also U3.1 (GND)
- net MISO: now also U3.7 (MISO)
- net MOSI: now also U3.6 (MOSI)
- net NSS: now also U3.4 (~{CSN})
- net SCLK: now also U3.5 (SCK)
- net RFM0 renamed CE
- net CE: now also U3.8 (IRQ)
- net RFMreset renamed IRQ
- net IRQ: now also U3.3 (CE)
Other:
- note added: "nrf transiever"
- note removed: "RFM69HCW 915MHz transceiver"
- moved on the sheet: C1
